File: Marmoset_Breakout/Marmoset_Breakout.sch (KiCad schematic (older format))
At the start: 43 parts, among them P1 CONN_01X05, P2 CONN_01X04, P3 CONN_01X04, Q1 DTC114YKA, Q2 DTC114YKA, U1 CONN_CHIP1, U2 CONN_DISPLAY, U3 PCF8563T/5, U4 CONN_AUDIO, U5 PAM8302A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

Commit message: Fixed unconnected LCD Power Enable signal. Fixed audio schematic and redid layout accordingly.
Parts:
- removed P2: CONN_01X04, Pin_Headers:Pin_Header_Straight_1x04, symbol CONN_01X04
- removed Q1: DTC114YKA, Marmoset:SOT-23-3, symbol DTC114YKA
- added P2: CONN_01X05, Pin_Headers:Pin_Header_Straight_1x05, symbol CONN_01X05
Connections:
- net +3V3_A: now also P2.1 (P1)
- net +3V3_D: now also U2.40 (VDDI), U2.41 (VDDI), U2.42 (VCI)
- net GND_A: now also P2.5 (P5); no longer C4.2
- net HP_L: now also P2.4 (P4); no longer VR1.3
- net HP_R: now also VR1.3, P2.3 (P3)
- net at R8.1, U4.4: no longer C7.2, VR1.1
- new net HP_GND: C4.2, C7.2, P2.2 (P2), VR1.1
Other:
- moved on the sheet: BT1, C10, C11, C12, C2, C3, C4, C5, C6, C7, C8, C9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

Commit message: Fixed Shutdown circuit for audio amp to use negative logic (as specified in datasheet) Fixed debouncing circuit for headphone ground pin. Added another pin to audio board to allow me to choose voltage for amplifier for testing. (I'm pretty sure it should be 3.3V but this will allow me to be sure) Updated layout accordingly.
Parts:
- removed P2: CONN_01X05, Pin_Headers:Pin_Header_Straight_1x05, symbol CONN_01X05
- added P2: CONN_01X06, Pin_Headers:Pin_Header_Straight_1x06, symbol CONN_01X06
Connections:
- net +3V3_A: now also R9.2, P2.2 (P2); no longer C10.2, R10.2, U5.6 (VDD)
- net GND_A: now also C4.2, R10.1, P2.6 (P6); no longer R9.2
- net HP_GND: now also R8.1, U4.4, P2.3 (P3); no longer C4.2
- net HP_L: now also P2.5 (P5)
- net HP_R: now also P2.4 (P4)
- net at C8.1, U4.5, U5.1 (SD): now also R10.2; no longer R10.1
- new net V_AMP: C10.2, P2.1 (P1), U5.6 (VDD)
Other:
- note added: "I had to add my own \naudio jack because \nthe NTC guys didn't\ngive me access to the HP\nDetect signal."
- note removed: "I had to add my own audio jack\nbecause the NTC guys didn't\ngive me access to the HP\nDetect signal."
- moved on the sheet: C2, C3, C4, C8, R10, R6, R7, R8, R9

Commit message: Changed Speaker used and updated BOM/Schematic.
Parts:
- BT1: footprint Marmoset:BU2032-SM -> Marmoset:SMTU2032-LF
Changed lines of the file:
@@
 F 0 "BT1" H 7200 5250 50  0000 C CNN
 F 1 "BATT_2032" H 7200 4860 50  0000 C CNN
-F 2 "Marmoset:BU2032-SM" H 7200 5050 60  0001 C CNN
+F 2 "Marmoset:SMTU2032-LF" H 7200 5050 60  0001 C CNN
 F 3 "http://www.digikey.com/product-detail/en/BU2032SM-BT-GTR/BU2032SM-BT-GTR-ND/2439521" H 7200 5700 60  0001 C CNN
 F 4 "0.60" H 8050 5600 60  0001 C CNN "Price"
